File: placa_IoT/RF.kicad_sch (KiCad schematic)
At the start: 0 parts

Commit message: Antena add
Parts:
- added ANT2: I-PEX MHF I, antennas:IPEX_MHF_I, symbol antennas:IPEX_MHF_I
- added C22, C23, C24: NC, Capacitor_SMD:C_0402_1005Metric, symbol Device:C
- added R10, R11, R8, R9: 22 Ohm, Resistor_SMD:R_0402_1005Metric, symbol Device:R
- added R12: OR, Resistor_SMD:R_0402_1005Metric, symbol Device:R
- added U5: T-SX1262, ic_control:MODULE_T_SX1262, symbol ic_control:T_SX1262
Connections:
- new net: R11.1, U5.9 (BUSY)
- new net: C23.2, C24.1, R12.2
- new net: ANT2.1 (In), R12.1
- new net: R9.1, U5.13 (NC)
- new net: R8.1, U5.14 (DIO3)
- new net: R10.1, U5.10 (DIO1)
- new net: C22.2, C24.2, U5.16 (ANT)
- new net +3.3V: U5.12 (3.3V)
- new net GND: ANT2.2 (Ext), C22.1, C23.1, U5.1 (GND), U5.15 (GND), U5.8 (GND)
- new net IO3: U5.7 (MISO)
- new net IO33: R10.2
- new net IO34: R11.2
- new net IO36: U5.2 (NC)
- new net IO5: U5.5 (SCK)
- new net IO6: U5.6 (MOSI)
- new net IO7: U5.4 (NSS)
- new net IO8: U5.3 (NRESET)
- new net IO9: U5.11 (NC)
- new net LORA_RX: R8.2
- new net LORA_TX: R9.2

Commit message: No conectar elementos
Parts:
- C22, C23: now not fitted
Changed lines of the file:
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@@
 		(on_board yes)
 		(in_pos_files yes)
-		(dnp no)
+		(dnp yes)
 		(fields_autoplaced yes)
 		(property "Reference" "C23"
@@
 		(on_board yes)
 		(in_pos_files yes)
-		(dnp no)
+		(dnp yes)
 		(fields_autoplaced yes)
 		(property "Reference" "C22"
