File: placa_IoT/bateria.kicad_sch (KiCad schematic)
At the start: 0 parts

Commit message: Batería completed
Parts:
- added C25, C27: 10 uF, Capacitor_SMD:C_0402_1005Metric, symbol Device:C
- added C26, C28: 100 nF, Capacitor_SMD:C_0402_1005Metric, symbol Device:C
- added D1, D3: SS34, Diode_SMD:D_SMA, symbol Diode:SS34
- added D2: DZ 5.6 V, Diode_SMD:D_SOD-123, symbol Device:D_Zener
- added D4: LED RED, LED_SMD:LED_0402_1005Metric, symbol Device:LED
- added D5: LED BLUE, LED_SMD:LED_0402_1005Metric, symbol Device:LED
- added J3: B2B-PH-K-S(LF)(SN), connectors:CONN_THT_MV_JST_P2.00MM_P2, symbol connectors:CONN_THT_MV_JST_P2.00MM_P2
- added J5: 620102131822, connectors:CONN_SMT_MH_SH_P2.00MM_P2, symbol connectors:CONN_SMT_MH_SH_P2.00MM_P2
- added Q1, Q2: Q_PMOS, Package_TO_SOT_SMD:SOT-23, symbol Device:Q_PMOS
- added R13: 499 Ohm, Resistor_SMD:R_0402_1005Metric, symbol Device:R
- added R14, R15: 100 kOhm, Resistor_SMD:R_0402_1005Metric, symbol Device:R
- added R16, R17: 1 kOhm, Resistor_SMD:R_0402_1005Metric, symbol Device:R
- added R18: 2 kOhm, Resistor_SMD:R_0402_1005Metric, symbol Device:R
- added R19: 0, Resistor_SMD:R_0402_1005Metric, symbol Device:R
- added R20, R21: 100 kOhm 1%, Resistor_SMD:R_0402_1005Metric, symbol Device:R
- added SW4: SW_SPDT, symbol Switch:SW_SPDT
- added U6: CN3065, ic_power:DFN-8-1EP_3x3mm_P0.5mm_EP1.66x2.38mm, symbol ic_power:CN3065
Connections:
- new net: D5.1 (K), U6.7 (~{CHRG})
- new net: D5.2 (A), R17.1
- new net: C25.1, C26.1, D3.1 (K), Q2.S, R16.2, R17.2, U6.4 (VIN)
- new net: D4.1 (K), U6.6 (~{DONE})
- new net: D4.2 (A), R16.1
- new net: R19.2, U6.1 (TEMP)
- new net: R18.2, U6.2 (ISET)
- new net: D1.1 (K), Q1.S, SW4.2 (B)
- new net +5V: SW4.1 (A)
- new net DBUS: D3.2 (A), Q2.G
- new net GND: C25.2, C26.2, C27.2, C28.2, D2.2 (A), J3.1 (Pin_1), J5.2 (Pin_2), R13.1, R15.1, R18.1, R19.1, R21.1, U6.3 (GND), U6.9 (GND)
- new net IO1: C28.1, R20.1, R21.2
- new net IO4: R14.1, R15.2
- new net V SOLAR: D2.1 (K), J3.2 (Pin_2), Q2.D, R14.2
- new net VBAT: C27.1, J5.1 (Pin_1), Q1.D, R20.2, U6.5 (BAT), U6.8 (FB)
- new net VBUS: D1.2 (A), Q1.G, R13.2
- no-connect marks 0 -> 3

Commit message: USB completed
Changed lines of the file:
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@@
 		(dnp no)
 		(property "Reference" "J3"
-			(at 20.32 88.9 0)
+			(at 24.13 95.885 0)
 			(show_name no)
 			(do_not_autoplace yes)
@@
 		)
 		(property "Value" "B2B-PH-K-S(LF)(SN)"
-			(at 20.32 91.44 0)
+			(at 34.925 98.425 0)
 			(show_name no)
 			(do_not_autoplace yes)

Commit message: Falta unir pines
Changed lines of the file:
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@@
 	)
 	(hierarchical_label "IO1"
-		(shape bidirectional)
+		(shape output)
 		(at 246.38 132.08 0)
 		(effects

Commit message: Errores placa solucionados
Parts:
- SW4: footprint (none) -> Button_Switch_THT:SW_Slide_SPDT_Angled_CK_OS102011MA1Q
Connections:
- net DBUS: now also Q2.1 (G); no longer Q2.G
- net V SOLAR: now also Q2.3 (D); no longer Q2.D
- net VBAT: now also Q1.3 (D); no longer Q1.D
- net VBUS: now also Q1.1 (G); no longer Q1.G
- net at C25.1, C26.1, D3.1 (K)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: now also Q2.2 (S); no longer Q2.S
- net at D1.1 (K), SW4.2 (B): now also Q1.2 (S); no longer Q1.S
Changed lines of the file:
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@@
 			)
 		)
-		(property "Footprint" ""
+		(property "Footprint" "Button_Switch_THT:SW_Slide_SPDT_Angled_CK_OS102011MA1Q"
 			(at 64.77 57.15 0)
 			(hide yes)
@@
 	)
 	(symbol
+		(lib_name "Q_PMOS_1")
 		(lib_id "Device:Q_PMOS")
 		(at 63.5 93.98 90)
@@
 			)
 		)
-		(pin "G"
-		)
-		(pin "D"
-		)
-		(pin "S"
+		(pin "2"
+		)
+		(pin "3"
+		)
+		(pin "1"
 		)
 		(instances
@@
 			)
 		)
-		(pin "G"
-		)
-		(pin "D"
-		)
-		(pin "S"
-		)
-		(instances
+		(pin "3"
+		)
+		(pin "2"
+		)
+		(pin "1"
+		)
+		(instances
